File: KiCad/Solar_Tracker.sch (KiCad schematic (older format))
At the start: 134 parts, among them J1 +48V_IN, J10 HOLE, J11 HOLE, J12 HOLE, J13 HOLE, J14 ELJMP, J2 USB_OTG, J3 EL, J4 CONN_01X05, J5 CONN_02X03, J6 GPIO, J7 AZJMP, J8 AZ, J9 CONN_01X03, Q1 BUK9M42-60E, Q2 BUK9M42-60E, Q3 BUK9M42-60E, Q4 BUK9M42-60E, Q5 BUK9M42-60E, Q6 BUK9M42-60E, Q7 BUK9M42-60E, Q8 BUK9M42-60E, SW1 SWITCH, U1 MER1S4805SC, U10 TLP291, U11 75LBC182, U12 A4927, U2 A4927, U3 ATMEGA32U4-AU, U4 A4927, U5 A4927, U6 MER1S4805SC, U7 TLP291, U8 TLP291, U9 TLP291, Y1 16MHz

Commit message: Updated capacitor symbol in schematic, updated linkings between components and symbols
Parts:
- removed C9: 10000u, Capacitors_THT:CP_Radial_D22.0mm_P10.00mm_SnapIn, symbol CP
- added C9: 10000u, symbol SNAP_CAP
Connections:
- wire segments 422 -> 549

Commit message: Added mounting hole footprint, tied to hole symbol
Parts:
- C9: footprint (none) -> SOLAR_TRACKER:vnd_cap
- D14, D7, D8, D9: footprint (none) -> SOLAR_TRACKER:tvs_quad
- D2: footprint (none) -> SOLAR_TRACKER:tvs_usb
- J10, J11, J12, J13: footprint (none) -> SOLAR_TRACKER:M3
- U1, U6: footprint (none) -> SOLAR_TRACKER:5v_iso
- Y1: footprint (none) -> SOLAR_TRACKER:resonator

Commit message: Work on grouping components
Parts:
- Q1, Q2, Q3, Q4, Q5, Q6, Q7, Q8: footprint Solar:nFET -> SOLAR_TRACKER:nFET
Changed lines of the file:
@@
 F 0 "Q8" H 15450 3950 60  0000 C CNN
 F 1 "BUK9M42-60E" H 15600 3550 60  0000 C CNN
-F 2 "Solar:nFET" V 15300 3450 60  0001 C CNN
+F 2 "SOLAR_TRACKER:nFET" V 15300 3450 60  0001 C CNN
 F 3 "" V 15300 3450 60  0001 C CNN
 	1    15250 3750
@@
 F 0 "Q7" H 14250 3950 60  0000 C CNN
 F 1 "BUK9M42-60E" H 14400 3550 60  0000 C CNN
-F 2 "Solar:nFET" V 14100 3450 60  0001 C CNN
+F 2 "SOLAR_TRACKER:nFET" V 14100 3450 60  0001 C CNN
 F 3 "" V 14100 3450 60  0001 C CNN
 	1    14050 3750
@@
 F 0 "Q6" H 11400 3950 60  0000 C CNN
 F 1 "BUK9M42-60E" H 11550 3550 60  0000 C CNN
-F 2 "Solar:nFET" V 11250 3450 60  0001 C CNN
+F 2 "SOLAR_TRACKER:nFET" V 11250 3450 60  0001 C CNN
 F 3 "" V 11250 3450 60  0001 C CNN
 	1    11200 3750
@@
 F 0 "Q5" H 10200 3950 60  0000 C CNN
 F 1 "BUK9M42-60E" H 10350 3550 60  0000 C CNN
-F 2 "Solar:nFET" V 10050 3450 60  0001 C CNN
+F 2 "SOLAR_TRACKER:nFET" V 10050 3450 60  0001 C CNN
 F 3 "" V 10050 3450 60  0001 C CNN
 	1    10000 3750
@@
 F 0 "Q4" H 7400 3950 60  0000 C CNN
 F 1 "BUK9M42-60E" H 7550 3550 60  0000 C CNN
-F 2 "Solar:nFET" V 7250 3450 60  0001 C CNN
+F 2 "SOLAR_TRACKER:nFET" V 7250 3450 60  0001 C CNN
 F 3 "" V 7250 3450 60  0001 C CNN
 	1    7200 3750
@@
 F 0 "Q3" H 6200 3950 60  0000 C CNN
 F 1 "BUK9M42-60E" H 6350 3550 60  0000 C CNN
-F 2 "Solar:nFET" V 6050 3450 60  0001 C CNN
+F 2 "SOLAR_TRACKER:nFET" V 6050 3450 60  0001 C CNN
 F 3 "" V 6050 3450 60  0001 C CNN
 	1    6000 3750
@@
 F 0 "Q2" H 3400 3950 60  0000 C CNN
 F 1 "BUK9M42-60E" H 3550 3550 60  0000 C CNN
-F 2 "Solar:nFET" V 3250 3450 60  0001 C CNN
+F 2 "SOLAR_TRACKER:nFET" V 3250 3450 60  0001 C CNN
 F 3 "" V 3250 3450 60  0001 C CNN
 	1    3200 3750
@@
 F 0 "Q1" H 2200 3950 60  0000 C CNN
 F 1 "BUK9M42-60E" H 2350 3550 60  0000 C CNN
-F 2 "Solar:nFET" V 2050 3450 60  0001 C CNN
+F 2 "SOLAR_TRACKER:nFET" V 2050 3450 60  0001 C CNN
 F 3 "" V 2050 3450 60  0001 C CNN
 	1    2000 3750

Commit message: Updated schematic to use Nano, added Nano part
Parts:
- removed C1, C11, C12, C13, C14: 1u, Capacitors_SMD:C_1206_HandSoldering, symbol C
- removed D14, D8: TVS_x4, SOLAR_TRACKER:tvs_quad, symbol TVS_x4
- removed D2: TVS_USB, SOLAR_TRACKER:tvs_usb, symbol TVS_USB
- removed J2: USB_OTG, Connectors:USB_Micro-B, symbol USB_OTG
- removed J5: CONN_02X03, Pin_Headers:Pin_Header_Straight_2x03_Pitch2.54mm, symbol CONN_02X03
- removed J6: GPIO, Connectors_Phoenix:PhoenixContact_GMSTBA-G_08x7.50mm_Angled, symbol CONN_01X08
- removed R2: 1K, Resistors_SMD:R_1206_HandSoldering, symbol R
- removed R3, R4: 22, Resistors_SMD:R_1206_HandSoldering, symbol R
- removed SW1: SWITCH, Buttons_Switches_SMD:SW_SPST_B3S-1000, symbol SWITCH
- removed U3: ATMEGA32U4-AU, Housings_QFP:TQFP-44_10x10mm_Pitch0.8mm, symbol ATMEGA32U4-AU
- removed Y1: 16MHz, SOLAR_TRACKER:resonator, symbol Resonator
- added J6, J?: GPIO, Connectors_Phoenix:PhoenixContact_GMSTBA-G_02x7.50mm_Angled, symbol CONN_01X02
- added U?: Nano, symbol Nano
- U12, U2, U4, U5: symbol A4927 -> A4927-RESCUE-Solar_Tracker
Connections:
- net +5V: now also U?.30 (VIN)
- net AZRTE: now also U?.15 (PB4)
- net ELRTE: now also U?.16 (PB5)
- net EN: now also U?.9 (PD6)
- net Earth: now also U12.P (PAD), U2.P (PAD), U4.P (PAD), U5.P (PAD), U?.29 (GND), U?.4 (GND); no longer U12.25 (PAD), U2.25 (PAD), U4.25 (PAD), U5.25 (PAD)
- net ISO_PWR_DET: now also U?.10 (PD7)
- net RX: now also U?.2 (RXD)
- net TX: now also U?.1 (TXD)
- net at C2.1: now also U?.18 (AREF)
- net D4 renamed C0
- net C0: now also J6.1 (P1), U?.19 (PC0)
- net D5 renamed C1
- net C1: now also J6.2 (P2), U?.20 (PC1)
- net D6 renamed C2
- net C2: now also J?.1 (P1), U?.21 (PC2)
- net D7 renamed C3
- net C3: now also J?.2 (P2), U?.22 (PC3)
- net E2 renamed RLED
- net RLED: now also U?.24 (PC5)
- net E6 renamed TLED
- net TLED: now also U?.23 (PC4)
- net MISO renamed AZBL
- net AZBL: now also U?.6 (PD3)
- net MOSI renamed AZBH
- net AZBH: now also U?.5 (PD2)
- net PB0 renamed AZFH
- net AZFH: now also U?.7 (PD4)
- net PB1 renamed AZFL
- net AZFL: now also U?.8 (PD5)
- net PB4 renamed ELFH
- net ELFH: now also U?.13 (PB2)
- net PB5 renamed ELFL
- net ELFL: now also U?.14 (PB3)
- net PB6 renamed ELBH
- net ELBH: now also U?.11 (PB0)
- net PB7 renamed ELBL
- net ELBL: now also U?.12 (PB1)
- new net A6: U?.25 (ADC6)
- new net A7: U?.26 (ADC7)
Other:
- moved on the sheet: C10, C2, D9

Commit message: Updated annotation
Parts:
- gave numbers to parts that had none: 2
- renumbered C10 to C1, C9 to C10, C15 to C11, C16 to C12, C17 to C13, C18 to C14, C19 to C15, C20 to C16, C21 to C17, C22 to C18, C23 to C19, C24 to C20, C25 to C21, C37 to C22, C27 to C23, C28 to C24, C29 to C25, C30 to C26, C31 to C27, C32 to C28, C33 to C29, C34 to C30, C35 to C31, C26 to C32, C36 to C8, C8 to C9, D13 to D10, D6 to D11, D15 to D12, D3 to D2, D4 to D3, D5 to D4, D7 to D5, D9 to D6, D10 to D7, D11 to D8, D12 to D9, J7 to J10, J14 to J11, J8 to J12, J9 to J13, J10 to J2, J11 to J3, J3 to J4, J12 to J5, J13 to J6, J4 to J7, J6 to J8, R13 to R10, R14 to R11, R15 to R12, R44 to R13, R16 to R14, R17 to R15, R18 to R16, R19 to R17, R20 to R18, R21 to R19, R5 to R2, R22 to R20, R23 to R21, R24 to R22, R25 to R23, R26 to R24, R27 to R25, R28 to R26, R29 to R27, R30 to R28, R31 to R29, R6 to R3, R32 to R30, R33 to R31, R34 to R32, R35 to R33, R36 to R34, R37 to R35, R38 to R36, R39 to R37, R40 to R38, R41 to R39, R7 to R4, R42 to R40, R43 to R41, R8 to R5, R9 to R6, R10 to R7, R11 to R8, R12 to R9

Commit message: Fixing library issues
Parts:
- removed U12, U2, U4, U5: A4927, Housings_SSOP:ST_PowerSSO-24_SlugDown_ThermalVias, symbol A4927-RESCUE-Solar_Tracker
- added U? (x4): A4927, symbol A4927
Connections:
- net +48V: now also U?.23 (VBB), U?.23 (VBB), U?.23 (VBB), U?.23 (VBB), U?.24 (VBRG), U?.24 (VBRG), U?.24 (VBRG), U?.24 (VBRG)
- net AZBH: now also U?.5 (HS)
- net AZBL: now also U?.6 (LSn)
- net AZFH: now also U?.5 (HS)
- net AZFL: now also U?.6 (LSn)
- net AZ_B: now also U?.18 (S)
- net AZ_F: now also U?.18 (S)
- net ELBH: now also U?.5 (HS)
- net ELBL: now also U?.6 (LSn)
- net ELFH: now also U?.5 (HS)
- net ELFL: now also U?.6 (LSn)
- net EL_B: now also U?.18 (S)
- net EL_F: now also U?.18 (S)
- net Earth: now also U?.1 (GND), U?.1 (GND), U?.1 (GND), U?.1 (GND), U?.25 (PAD), U?.25 (PAD), U?.25 (PAD), U?.25 (PAD)
- net at C27.2, D10.2 (A), Q7.1 (S)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: now also U?.15 (LSS)
- net at R39.2: now also U?.16 (GL)
- net at R40.2: now also U?.17 (GH)
- net at C29.2: now also U?.19 (C)
- net at C24.1: now also U?.20 (VREG)
- net at C32.1: now also U?.21 (CP2)
- net at C32.2: now also U?.22 (CP1)
- net at R41.2: now also U?.3 (ENABLE), U?.4 (RESETn)
- net at C18.2, D7.2 (A), Q5.1 (S)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: now also U?.15 (LSS)
- net at R17.2: now also U?.16 (GL)
- net at R22.2: now also U?.17 (GH)
- net at C19.2: now also U?.19 (C)
- net at C16.1: now also U?.20 (VREG)
- net at C20.1: now also U?.21 (CP2)
- net at C20.2: now also U?.22 (CP1)
- net at R24.2: now also U?.3 (ENABLE), U?.4 (RESETn)
- net at C13.2, D4.2 (A), Q3.1 (S)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: now also U?.15 (LSS)
- net at R10.2: now also U?.16 (GL)
- net at R11.2: now also U?.17 (GH)
- net at C14.2: now also U?.19 (C)
- net at C11.1: now also U?.20 (VREG)
- net at C15.1: now also U?.21 (CP2)
- net at C15.2: now also U?.22 (CP1)
- net at R12.2: now also U?.3 (ENABLE), U?.4 (RESETn)
- net at C5.2, D1.2 (A), Q1.1 (S)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: now also U?.15 (LSS)
- net at R2.2: now also U?.16 (GL)
- net at R3.2: now also U?.17 (GH)
- net at C7.2: now also U?.19 (C)
- net at C3.1: now also U?.20 (VREG)
- net at C9.1: now also U?.21 (CP2)
- net at C9.2: now also U?.22 (CP1)
- net at R4.2: now also U?.3 (ENABLE), U?.4 (RESETn)

Commit message: Added nano footprint
Parts:
- U12, U2, U4, U5: renamed from U?; footprint (none) -> Housings_SSOP:ST_PowerSSO-24_SlugDown_ThermalVias
- U3: footprint (none) -> SOLAR_TRACKER:nano

Commit message: Updated netlist in pcb
Parts:
- U10, U7, U8, U9: footprint Housings_DIP:DIP-4_W7.62mm_SMD -> SOLAR_TRACKER:opto
