File: KiCad/_autosave-Solar_Tracker.kicad_pcb (KiCad board)
At the start: 2 copper layers, 87.6 x 184.2 mm, 120 parts, among them J1 +48V_IN, J10 AZJMP, J11 ELJMP, J12 AZ, J13 CONN_01X03, J2 HOLE, J3 HOLE, J4 EL, J5 HOLE, J6 HOLE, J7 CONN_01X05, J8 GPIO, J9 GPIO, Q1 BUK9M42-60E, Q2 BUK9M42-60E, Q3 BUK9M42-60E, Q4 BUK9M42-60E, Q5 BUK9M42-60E, Q6 BUK9M42-60E, Q7 BUK9M42-60E, Q8 BUK9M42-60E, U1 MER1S4805SC, U10 TLP291, U11 75LBC182, U12 A4927, U2 A4927, U3 Nano, U4 A4927, U5 A4927, U6 MER1S4805SC, U7 TLP291, U8 TLP291, U9 TLP291

Commit message: attempt 1 at motor layout
Parts:
- moved C16 46.0 mm to (102.1, 162.1), turned to 270 degrees
- moved C17 44.4 mm to (102.4, 147.1), turned to 270 degrees
- moved C19 42.7 mm to (102.1, 155.2), turned to 270 degrees
- moved C20 38.5 mm to (107.2, 158.2)
- moved R16 27.9 mm to (119.4, 159.8), turned to 270 degrees
- moved D7 15.2 mm to (119.4, 152.9), turned to 90 degrees
- moved Q6 7.42 mm to (106.2, 150.4)
- moved C18 5.85 mm to (118.9, 143.8), turned to 270 degrees
- moved R22 2.30 mm to (111.8, 151.4)
- moved Q5 2.05 mm to (112.3, 147.6)
- moved R17 2.05 mm to (114.3, 151.6)
Routing:
- net +48V: track 0.00 -> 72.4 mm
- net AZ_B: track 0.00 -> 25.7 mm
- net Net-(C19-Pad2): track 0.00 -> 12.3 mm
- net Net-(C16-Pad1): track 0.00 -> 12.1 mm
- net Net-(R22-Pad2): track 0.00 -> 5.91 mm
- net Net-(R17-Pad2): track 0.00 -> 5.39 mm

Commit message: more updates
Parts:
- moved C29 215.8 mm to (190.8, 157.0)
- moved Q7 207.3 mm to (190.8, 162.6), turned to 270 degrees
- moved U12 185.2 mm to (179.8, 153.9)
- moved R41 180.0 mm to (178.1, 127.3)
- moved Q8 179.9 mm to (165.9, 141.7)
- moved R39 138.6 mm to (190.8, 159.5), turned to 180 degrees
- moved R30 133.7 mm to (186.4, 126.7)
- moved C32 124.0 mm to (190.8, 151.6)
- moved R40 103.5 mm to (176.8, 121.7)
- moved C25 87.7 mm to (172.2, 128.5)
- moved C27 87.1 mm to (184.9, 116.3)
- moved C24 78.8 mm to (190.8, 154.2)
- moved D10 54.7 mm to (184.9, 120.7)
Routing:
- net Net-(C29-Pad2): track 0.00 -> 10.5 mm
- net Net-(C32-Pad2): track 0.00 -> 10.4 mm
- net Net-(C18-Pad2): track 0.00 -> 8.38 mm
- net Net-(R39-Pad2): track 0.00 -> 7.11 mm
- net Net-(C24-Pad1): track 0.00 -> 4.89 mm
- net Net-(R24-Pad2): track 0.00 -> 4.69 mm
- net Net-(C32-Pad1): track 0.00 -> 4.11 mm
Other:
- board text added: "Notes: How does AZ get out with power in a line?"
