File: KiCad/Solar_Tracker.kicad_pcb (KiCad board)
At the start: 2 copper layers, 160 x 100 mm, 116 parts, among them J1 +48V, J10 AZJMP, J11 ELJMP, J12 AZ, J13 CONN_01X03, J2 HOLE, J3 HOLE, J4 EL, J5 HOLE, J6 HOLE, J7 CONN_01X05, J8 GPIO, J9 GPIO, Q1 BUK9M42-60E, Q2 BUK9M42-60E, Q3 BUK9M42-60E, Q4 BUK9M42-60E, Q5 BUK9M42-60E, Q6 BUK9M42-60E, Q7 BUK9M42-60E, Q8 BUK9M42-60E, U1 MER1S4805SC, U10 TLP291, U11 75LBC182, U12 A4927, U2 A4927, U3 Nano, U4 A4927, U5 A4927, U6 MER1S4805SC, U7 TLP291, U8 TLP291, U9 TLP291

Commit message: Silky smooth ;)
Other:
- board text added: "+"
- board text added: "+ RED"
- board text added: "+48V"
- board text added: "+48V IN"
- board text added: "-"
- board text added: "- BLK"
- board text added: "5V"
- board text added: "AZIMUTH MOTOR"
- board text added: "AZ_B"
- board text added: "AZ_F"
- board text added: "BARE"
- board text added: "BLK"
- board text added: "C0"
- board text added: "C1"
- board text added: "C2"
- board text added: "C3"
- board text added: "CWRU CSE EECS 2017 W. Nourse D. G. Parikh P. Van Rooy Advisor: Dr. G. Lee"
- board text added: "Documentation Available At: https://github.com/wnourse05/Lake_Metroparks_Farmpark_Solar_Tracker"
- board text added: "ELEVATION MOTOR"
- board text added: "EL_B"
- board text added: "EL_F"
- board text added: "GND"
- board text added: "GRN"
- board text added: "ISO 5V"
- board text added: "RED"
- board text added: "RS485"
- board text added: "RX"
- board text added: "SENSOR"
- board text added: "TX"
- board text added: "USB GOES HERE"
- board text added: "WHT"
- board text added: "YLW"
Changed lines of the file:
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@@
     (area 11.924999 11.924999 172.075001 112.075001)
     (thickness 1.6)
-    (drawings 4)
+    (drawings 39)
     (tracks 901)
     (zones 0)
@@
     (tags "LED 1206")
     (attr smd)
-    (fp_text reference D3 (at 0 -1.85 180) (layer F.SilkS)
+    (fp_text reference D3 (at 0 1.905 180) (layer F.SilkS)
       (effects (font (size 1 1) (thickness 0.15)))
     )
@@
     (tags "LED 1206")
     (attr smd)
-    (fp_text reference D4 (at 0 -1.85 270) (layer F.SilkS)
+    (fp_text reference D4 (at -3.2195 2.0625 270) (layer F.SilkS)
       (effects (font (size 1 1) (thickness 0.15)))
     )
@@
     (tags "LED 1206")
     (attr smd)
-    (fp_text reference D11 (at -0.635 -2.1336 180) (layer F.SilkS)
+    (fp_text reference D11 (at 0 -1.778 180) (layer F.SilkS)
       (effects (font (size 1 1) (thickness 0.15)))
     )
@@
     (tags "resistor 1206")
     (attr smd)
-    (fp_text reference L2 (at 0 -2.3 270) (layer F.SilkS)
+    (fp_text reference L2 (at -0.127 1.905 270) (layer F.SilkS)
       (effects (font (size 1 1) (thickness 0.15)))
     )
@@
     (tags "resistor 1206")
     (attr smd)
-    (fp_text reference R5 (at -0.2032 2.159 270) (layer F.SilkS)
+    (fp_text reference R5 (at -2.921 2.032 270) (layer F.SilkS)
       (effects (font (size 1 1) (thickness 0.15)))
     )
@@
     (tags "resistor 1206")
     (attr smd)
-    (fp_text reference R25 (at 0.2286 -2.921 270) (layer F.SilkS)
+    (fp_text reference R25 (at 0 2.032 270) (layer F.SilkS)
       (effects (font (size 1 1) (thickness 0.15)))
     )
@@
     (tags "resistor 1206")
     (attr smd)
-    (fp_text reference R26 (at -1.5494 2.3368 180) (layer F.SilkS)
+    (fp_text reference R26 (at 0.127 2.032 180) (layer F.SilkS)
       (effects (font (size 1 1) (thickness 0.15)))
     )
@@
     (tags "resistor 1206")
     (attr smd)
-    (fp_text reference R27 (at -2.0574 2.032 270) (layer F.SilkS)
+    (fp_text reference R27 (at 0 1.778 270) (layer F.SilkS)
       (effects (font (size 1 1) (thickness 0.15)))
     )
@@
     (tags "resistor 1206")
     (attr smd)
-    (fp_text reference R28 (at 0 -2.2098 180) (layer F.SilkS)
+    (fp_text reference R28 (at 0 1.524 180) (layer F.SilkS)
       (effects (font (size 1 1) (thickness 0.15)))
     )
@@
     (tags "resistor 1206")
     (attr smd)
-    (fp_text reference R29 (at 4.4704 -0.254 270) (layer F.SilkS)
+    (fp_text reference R29 (at 0 1.524 360) (layer F.SilkS)
       (effects (font (size 1 1) (thickness 0.15)))
     )
@@
     (tags "resistor 1206")
     (attr smd)
-    (fp_text reference R35 (at 0 -1.85 270) (layer F.SilkS)
+    (fp_text reference R35 (at -0.127 1.778 270) (layer F.SilkS)
       (effects (font (size 1 1) (thickness 0.15)))
     )
@@
     (tags "resistor 1206")
     (attr smd)
-    (fp_text reference R40 (at 0 -1.85 90) (layer F.SilkS)
+    (fp_text reference R40 (at 0 -1.524 90) (layer F.SilkS)
       (effects (font (size 1 1) (thickness 0.15)))
     )
@@
   (module SOLAR_TRACKER:opto (layer F.Cu)
     (at 53.848 72.136)
-    (fp_text reference U7 (at -2.3876 -1.0668 90) (layer F.SilkS)
+    (fp_text reference U7 (at -2.413 -0.127 90) (layer F.SilkS)
       (effects (font (size 1 1) (thickness 0.15)))
     )
@@
   (module SOLAR_TRACKER:opto (layer F.Cu)
     (at 48.514 72.136)
-    (fp_text reference U8 (at -2.5146 -1.2192 90) (layer F.SilkS)
+    (fp_text reference U8 (at -2.413 0 90) (layer F.SilkS)
       (effects (font (size 1 1) (thickness 0.15)))
     )
@@
   (module SOLAR_TRACKER:opto (layer F.Cu)
     (at 40.894 72.39 180)
-    (fp_text reference U9 (at -2.8702 0.9906 270) (layer F.SilkS)
+    (fp_text reference U9 (at 2.032 -0.127 270) (layer F.SilkS)
       (effects (font (size 1 1) (thickness 0.15)))
     )
@@
   (module SOLAR_TRACKER:opto (layer F.Cu)
     (at 36.576 72.39 180)
-    (fp_text reference U10 (at 2.5908 1.7272 270) (layer F.SilkS)
+    (fp_text reference U10 (at 2.286 -0.381 270) (layer F.SilkS)
       (effects (font (size 1 1) (thickness 0.15)))
     )
@@
   (module SOLAR_TRACKER:tvs_quad (layer F.Cu)
     (at 27.94 38.354 90)
-    (fp_text reference D5 (at 0.1524 -3.2766 90) (layer F.SilkS)
+    (fp_text reference D5 (at 0 2.667 90) (layer F.SilkS)
       (effects (font (size 1 1) (thickness 0.15)))
     )
@@
     (tags "LED 1206")
     (attr smd)
-    (fp_text reference D8 (at -0.5842 2.286 90) (layer F.SilkS)
+    (fp_text reference D8 (at -0.127 2.159 90) (layer F.SilkS)
       (effects (font (size 1 1) (thickness 0.15)))
     )
@@
     (tags "LED 1206")
     (attr smd)
-    (fp_text reference D9 (at 0.0762 -2.1082) (layer F.SilkS)
+    (fp_text reference D9 (at 0 1.905) (layer F.SilkS)
       (effects (font (size 1 1) (thickness 0.15)))
     )
@@
     (descr "Generic Phoenix Contact connector footprint for series: GMSTBA-G; number of pins: 05; pin pitch: 7.50mm; Angled || order number: 1766372 12A 630V")
     (tags "phoenix_contact connector GMSTBA_01x05_G_7.50mm")
-    (fp_text reference J7 (at 15 -3 270) (layer F.SilkS)
+    (fp_text reference J7 (at 11.069 -3.298 270) (layer F.SilkS)
       (effects (font (size 1 1) (thickness 0.15)))
     )
@@
     )
   )
+  (gr_text "Documentation Available At:\nhttps://github.com/wnourse05/Lake_Metroparks_Farmpark_Solar_Tracker" (at 159.766 108.077) (layer F.SilkS)
+    (effects (font (size 1.5 1.1) (thickness 0.275)) (justify right))
+  )
+  (gr_text "CWRU CSE EECS 2017\nW. Nourse\nD. G. Parikh\nP. Van Rooy\nAdvisor: Dr. G. Lee" (at 137.922 99.314) (layer F.SilkS)
+    (effects (font (size 1.5 1.5) (thickness 0.3)) (justify left))
+  )
+  (gr_text EL_F (at 78.105 46.736) (layer F.SilkS)
+    (effects (font (size 1.5 1.5) (thickness 0.3)))
+  )
+  (gr_text EL_B (at 167.386 38.227) (layer F.SilkS)
+    (effects (font (size 1.5 1.5) (thickness 0.3)))
+  )
+  (gr_text AZ_B (at 168.402 74.549) (layer F.SilkS)
+    (effects (font (size 1.5 1.5) (thickness 0.3)))
+  )
+  (gr_text AZ_F (at 76.581 85.344) (layer F.SilkS)
+    (effects (font (size 1.5 1.5) (thickness 0.3)))
+  )
+  (gr_text 5V (at 38.1 57.658) (layer F.SilkS)
+    (effects (font (size 1.5 1.5) (thickness 0.3)))
+  )
+  (gr_text TX (at 37.973 41.148) (layer F.SilkS)
+    (effects (font (size 1.5 1.5) (thickness 0.3)))
+  )
+  (gr_text RX (at 38.354 49.911) (layer F.SilkS)
+    (effects (font (size 1.5 1.5) (thickness 0.3)))
+  )
+  (gr_text +48V (at 88.9 17.78) (layer F.SilkS)
+    (effects (font (size 1.5 1.5) (thickness 0.3)))
+  )
+  (gr_text "ISO 5V" (at 68.834 86.741) (layer F.SilkS)
+    (effects (font (size 1.5 1.5) (thickness 0.3)))
+  )
+  (gr_text "USB GOES HERE" (at 53.848 25.146) (layer F.SilkS)
+    (effects (font (size 1.5 1.5) (thickness 0.3)))
+  )
+  (gr_text C2 (at 34.036 19.558) (layer F.SilkS)
+    (effects (font (size 1.5 1.5) (thickness 0.3)))
+  )
+  (gr_text C3 (at 54.356 19.304) (layer F.SilkS)
+    (effects (font (size 1.5 1.5) (thickness 0.3)))
+  )
+  (gr_text C0 (at 23.114 38.481) (layer F.SilkS)
+    (effects (font (size 1.5 1.5) (thickness 0.3)))
+  )
+  (gr_text C1 (at 22.86 24.765) (layer F.SilkS)
+    (effects (font (size 1.5 1.5) (thickness 0.3)))
+  )
+  (gr_text BARE (at 24.765 75.946) (layer F.SilkS)
+    (effects (font (size 1.5 1.5) (thickness 0.3)))
+  )
+  (gr_text BLK (at 24.257 68.326) (layer F.SilkS)
+    (effects (font (size 1.5 1.5) (thickness 0.3)))
+  )
+  (gr_text WHT (at 24.13 60.706) (layer F.SilkS)
+    (effects (font (size 1.5 1.5) (thickness 0.3)))
+  )
+  (gr_text GRN (at 24.892 53.086) (layer F.SilkS)
+    (effects (font (size 1.5 1.5) (thickness 0.3)))
+  )
+  (gr_text RED (at 24.765 45.974) (layer F.SilkS)
+    (effects (font (size 1.5 1.5) (thickness 0.3)))
+  )
+  (gr_text SENSOR (at 17.653 82.169) (layer F.SilkS)
+    (effects (font (size 1.5 1.5) (thickness 0.3)))
+  )
+  (gr_text GND (at 53.848 101.092) (layer F.SilkS)
+    (effects (font (size 1.5 1.5) (thickness 0.3)))
+  )
+  (gr_text - (at 45.466 100.965) (layer F.SilkS)
+    (effects (font (size 1.5 1.5) (thickness 0.3)))
+  )
+  (gr_text + (at 34.798 100.965) (layer F.SilkS)
+    (effects (font (size 1.5 1.5) (thickness 0.3)))
+  )
+  (gr_text RS485 (at 31.623 110.236) (layer F.SilkS)
+    (effects (font (size 1.5 1.5) (thickness 0.3)))
+  )
+  (gr_text "-\nBLK" (at 100.838 101.6) (layer F.SilkS)
+    (effects (font (size 1.5 1.5) (thickness 0.3)))
+  )
+  (gr_text "+\nRED" (at 80.264 101.473) (layer F.SilkS)
+    (effects (font (size 1.5 1.5) (thickness 0.3)))
+  )
+  (gr_text "+48V IN" (at 77.597 110.617) (layer F.SilkS)
+    (effects (font (size 1.5 1.5) (thickness 0.3)))
+  )
+  (gr_text "ELEVATION\nMOTOR" (at 117.856 25.781) (layer F.SilkS)
+    (effects (font (size 1.5 1.5) (thickness 0.3)))
+  )
+  (gr_text BLK (at 125.984 43.942 90) (layer F.SilkS)
+    (effects (font (size 1.5 1.5) (thickness 0.3)))
+  )
+  (gr_text RED (at 126.111 29.21 90) (layer F.SilkS)
+    (effects (font (size 1.5 1.5) (thickness 0.3)))
+  )
+  (gr_text "AZIMUTH\nMOTOR" (at 118.872 103.378) (layer F.SilkS)
+    (effects (font (size 1.5 1.5) (thickness 0.3)))
+  )
+  (gr_text YLW (at 127.635 84.328 90) (layer F.SilkS)
+    (effects (font (size 1.5 1.5) (thickness 0.3)))
+  )
+  (gr_text GRN (at 127.508 99.949 90) (layer F.SilkS)
+    (effects (font (size 1.5 1.5) (thickness 0.3)))
+  )
   (gr_line (start 172 112) (end 172 12) (angle 90) (layer Edge.Cuts) (width 0.15))
