File: KiCad/_saved_Solar_Tracker.sch (KiCad schematic (older format))
At the start: 123 parts, among them J1 +48V, J10 AZJMP, J11 ELJMP, J12 AZ, J13 CONN_01X03, J2 HOLE, J3 HOLE, J4 EL, J5 HOLE, J6 HOLE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

Commit message: Added expander to pcb
Parts:
- U13: footprint (none) -> Housings_SSOP:TSSOP-28_4.4x9.7mm_Pitch0.65mm
